Commit message: Change to joint trajectory controller

File: urdf/lc3_column.urdf.xacro (robot description, xacro)
@@ -7,7 +7,7 @@
         <visual>
             <geometry>
-                <box size="0.3 0.3 0.6"/>
+                <box size="0.3 0.3 0.1"/>
             </geometry>
-            <origin xyz="0 0 0.3" rpy="0 0 0"/>
+            <origin xyz="0 0 0.05" rpy="0 0 0"/>
             <material name="gray">
                 <color rgba="0.5 0.5 0.5 1"/>
@@ -16,7 +16,7 @@
         <collision>
             <geometry>
-                <box size="0.3 0.3 0.6"/>
+                <box size="0.3 0.3 0.1"/>
             </geometry>
-            <origin xyz="0 0 0.3" rpy="0 0 0"/>
+            <origin xyz="0 0 0.05" rpy="0 0 0"/>
         </collision>
         <inertial>
@@ -29,5 +29,5 @@
         <visual>
             <geometry>
-                <cylinder radius="0.05" length="0.5"/>
+                <box size="0.1 0.1 0.5"/>
             </geometry>
             <origin xyz="0 0 0.25" rpy="0 0 0"/>
@@ -38,5 +38,5 @@
         <collision>
             <geometry>
-                <cylinder radius="0.05" length="0.5"/>
+                <box size="0.1 0.1 0.5"/>
             </geometry>
             <origin xyz="0 0 0.25" rpy="0 0 0"/>

Commit message: Update URDF

File: urdf/lc3_column.urdf.xacro (robot description, xacro)
@@ -3,52 +3,70 @@
     <xacro:arg name="use_mock_hardware" default="false"/>
     <xacro:arg name="simulation" default="false"/>
-    <!-- Base link (fixed to world) -->
+    <!-- Base link-->
     <link name="base_link">
         <visual>
             <geometry>
-                <box size="0.3 0.3 0.1"/>
+                <box size="0.2 0.2 0.02"/>
             </geometry>
-            <origin xyz="0 0 0.05" rpy="0 0 0"/>
-            <material name="gray">
-                <color rgba="0.5 0.5 0.5 1"/>
+            <origin xyz="0 0 0.01" rpy="0 0 0"/>
+            <material name="light_gray">
+                <color rgba="0.7 0.7 0.7 1"/>
+            </material>
+        </visual>
+        <visual>
+            <geometry>
+                <box size="0.164 0.164 0.82"/>
+            </geometry>
+            <origin xyz="0 0 0.43" rpy="0 0 0"/>
+            <material name="light_gray">
+                <color rgba="0.7 0.7 0.7 1"/>
             </material>
         </visual>
         <collision>
             <geometry>
-                <box size="0.3 0.3 0.1"/>
+                <box size="0.164 0.164 0.84"/>
             </geometry>
-            <origin xyz="0 0 0.05" rpy="0 0 0"/>
+            <origin xyz="0 0 0.42" rpy="0 0 0"/>
         </collision>
         <inertial>
-            <mass value="5.0"/>
-            <inertia ixx="0.05" ixy="0.0" ixz="0.0" iyy="0.05" iyz="0.0" izz="0.05"/>
+            <mass value="10.0"/>
+            <inertia ixx="0.2" ixy="0.0" ixz="0.0" iyy="0.2" iyz="0.0" izz="0.03"/>
         </inertial>
     </link>
-    <!-- Column link (moving part) -->
+    <!-- Column link -->
     <link name="column_link">
         <visual>
             <geometry>
-                <box size="0.1 0.1 0.5"/>
+                <box size="0.148 0.148 0.80"/>
             </geometry>
-            <origin xyz="0 0 0.25" rpy="0 0 0"/>
-            <material name="silver">
-                <color rgba="0.75 0.75 0.75 1"/>
+            <origin xyz="0 0 0.40" rpy="0 0 0"/>
+            <material name="light_gray">
+                <color rgba="0.7 0.7 0.7 1"/>
+            </material>
+        </visual>
+        <visual>
+            <geometry>
+                <box size="0.129 0.129 0.84"/>
+            </geometry>
+            <origin xyz="0 0 0.82" rpy="0 0 0"/>
+            <material name="light_gray">
+                <color rgba="0.7 0.7 0.7 1"/>
             </material>
         </visual>
         <collision>
             <geometry>
-                <box size="0.1 0.1 0.5"/>
+                <box size="0.148 0.148 1.24"/>
             </geometry>
-            <origin xyz="0 0 0.25" rpy="0 0 0"/>
+            <origin xyz="0 0 0.62" rpy="0 0 0"/>
         </collision>
         <inertial>
-            <mass value="2.0"/>
-            <origin xyz="0 0 0.25" rpy="0 0 0"/>
-            <inertia ixx="0.05" ixy="0.0" ixz="0.0" iyy="0.05" iyz="0.0" izz="0.001"/>
+            <mass value="10.0"/>
+            <origin xyz="0 0 0.62" rpy="0 0 0"/>
+            <inertia ixx="0.12" ixy="0.0" ixz="0.0" iyy="0.12" iyz="0.0" izz="0.02"/>
         </inertial>
     </link>
     <!-- Prismatic joint for column -->
     <joint name="column_joint" type="prismatic">
-        <origin xyz="0 0 0.05" rpy="0 0 0"/>
+        <origin xyz="0 0 0" rpy="0 0 0"/>
         <parent link="base_link"/>
         <child link="column_link"/>
